File: AOS16 Double Buffer/word_buffer.kicad_sch (KiCad schematic)
At the start: 5 parts, among them IC4 SN74LVC16245ADGVR

Commit message: Completed double buffer first draft
Parts:
- C16: renamed from C13; value 0.1uF -> 0.01uF
- C17: renamed from C14; value 0.1uF -> 0.01uF
- C18: renamed from C15; value 0.1uF -> 0.01uF
- C19: renamed from C16; value 0.1uF -> 0.01uF
- IC3: renamed from IC4; footprint sn74lvc:SOP40P640X120-48N -> Package_SO:TSSOP-48_6.1x12.5mm_P0.5mm
Connections:
- net VCC renamed +3.3V
