File: AOS16 GPU/word_conn.kicad_sch (KiCad schematic)
At the start: 1 part, among them J5 Conn_02x08_Top_Bottom

Commit message: GPU PCB Design v1
Parts:
- renumbered J5 to J4
Changed lines of the file:
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@@
 		(dnp no)
 		(fields_autoplaced yes)
-		(property "Reference" "J5"
+		(property "Reference" "J4"
 			(at 70.485 53.34 0)
 			(effects
@@
 		(instances
 			(project "AOS16 GPU"
-				(path "/30867551-fb5e-4d50-9b6f-10252ea432a0/4f0cb423-5531-41a6-b585-748e68254428"
-					(reference "J7")
-					(unit 1)
-				)
 				(path "/30867551-fb5e-4d50-9b6f-10252ea432a0/66da1a66-ec4a-4320-afe7-b525d6b9c571"
-					(reference "J6")
+					(reference "J5")
 					(unit 1)
 				)
 				(path "/30867551-fb5e-4d50-9b6f-10252ea432a0/a0b27391-34e6-4924-9480-90aba22944d9"
-					(reference "J5")
+					(reference "J4")
 					(unit 1)
 				)
