File: AOS16 GPU/5bitdac.kicad_sch (KiCad schematic)
At the start: 15 parts, among them U22 MC33078

Commit message: updated gpu
Parts:
- removed R14: 13k, Resistor_SMD:R_0603_1608Metric, symbol Device:R
- removed R16: 75, Resistor_SMD:R_0603_1608Metric, symbol Device:R
- removed U22: MC33078, Package_SO:SOIC-8_3.9x4.9mm_P1.27mm, symbol Amplifier_Operational:MC33078
- added C1: 100 pF, Capacitor_SMD:C_0603_1608Metric, symbol Device:C
- added R37: 75, Resistor_SMD:R_0603_1608Metric, symbol Device:R
- added U22: LMH6642, Package_TO_SOT_SMD:SOT-23-5, symbol Amplifier_Operational:LMH6609MF
- R10, R12, R6, R8: value 10k -> 1k
- R11, R13, R4, R5, R7, R9: value 20k -> 2k
- R14: renamed from R15; value 5.1k -> 402; footprint Resistor_SMD:R_0603_1608Metric -> Resistor_SMD:R_0402_1005Metric
- renumbered C24 to C23
Connections:
- net +5V: now also C1.1, U22.5 (V+)
- net AOUT: now also R37.2
- net GND: now also C1.2, U22.2 (V-)
- net at R12.2, R13.1: now also R14.1, U22.3 (+)
- new net: R37.1, U22.1, U22.4 (-)
Other:
- moved on the sheet: C23, R14
