File: AOS16 GPU/AOS16 GPU.kicad_pcb (KiCad board)
At the start: 4 copper layers, 109 parts, among them J1 Conn_01x02, J2 Conn_01x01, J3 Conn_01x08, J4 DE15_Socket_HighDensity_Mount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, J5 Conn_02x08_Top_Bottom, J6 Conn_02x08_Top_Bottom, J7 Conn_02x08_Top_Bottom, U1 74AHC1GU04, U10 74LS30, U11 74LS30, U12 74HC00, U13 74AHC04, U14 74LS30, U15 74LS30, U16 74LS30, U17 74LS30, U18 74LS161, U19 74LS161, U2 74AHC1G14, U20 74LS161, U21 74HC00, U22 MC33078, U23 MC33078, U24 MC33078, U3 74AHC1G00, U4 74LS161, U5 74LS161, U6 74AHC04, U7 74AHC04, U8 74LS30, U9 74LS30, Y1 13.5 MHz

Commit message: GPU PCB Design v1
Parts:
- removed J6, J7: Conn_02x08_Top_Bottom, Connector_PinHeader_2.54mm:PinHeader_2x08_P2.54mm_Vertical
- removed R40: 13k, Resistor_SMD:R_0603_1608Metric
- removed R41: 5.1k, Resistor_SMD:R_0603_1608Metric
- removed R42: 75, Resistor_SMD:R_0603_1608Metric
- added C27: 0.1uF, Capacitor_SMD:C_0603_1608Metric, F.Cu at (106.8, 102.3)
- added U25: 74HC00, Package_SO:SOIC-14_3.9x8.7mm_P1.27mm, F.Cu at (96.3, 73.7)
- C1, C10, C11, C12, C13, C14, C15, C16, C17, C26, C4, J5, U14, U15, U16, U18, U19, U21: moved to B.Cu
- C5: value 0.1uF -> 50 pF
- C6: value 50 pF -> 0.1uF
- J3: value Conn_01x08 -> DE15_Socket_HighDensity_MountingHoles; footprint Connector_PinHeader_2.54mm:PinHeader_1x08_P2.54mm_Vertical -> Connector_Dsub:DSUB-15-HD_Socket_Horizontal_P2.29x1.90mm_EdgePinOffset3.03mm_Housed_MountingHolesOffset4.94mm
- J4: value DE15_Socket_HighDensity_MountingHoles -> Conn_02x08_Top_Bottom; footprint Connector_Dsub:DSUB-15-HD_Socket_Horizontal_P2.29x1.90mm_EdgePinOffset3.03mm_Housed_MountingHolesOffset4.94mm -> Connector_PinHeader_2.54mm:PinHeader_2x08_P2.54mm_Vertical; moved to B.Cu
- R10, R12, R6, R8: value 10k -> 1k; moved to B.Cu
- R11, R13, R4, R5, R7, R9: value 20k -> 2k; moved to B.Cu
- R14: value 13k -> 402
- R15: value 5.1k -> 2k
- R16, R29: value 75 -> 2k
- R17, R30: value 20k -> 1k
- R18, R20, R22, R24, R26, R31, R33, R35: value 20k -> 2k
- R19, R21, R23, R32, R34: value 10k -> 1k
- R2: footprint Resistor_SMD:R_0201_0603Metric -> Resistor_SMD:R_0603_1608Metric
- R25, R36: value 10k -> 402
- R27: value 13k -> 2k
- R28: value 5.1k -> 1k
- R37, R39: value 20k -> 75
- R38: value 10k -> 75
- U1: value 74AHC1GU04 -> 74AHC1G14
- U11: value 74LS30 -> 74HC00
- U12: value 74HC00 -> 74AHC04; moved to B.Cu
- U13: value 74AHC04 -> 74LS30; moved to B.Cu
- U17: value 74LS30 -> 74LS161; footprint Package_SO:SOIC-14_3.9x8.7mm_P1.27mm -> Package_SO:SOIC-16_3.9x9.9mm_P1.27mm; moved to B.Cu
- U2: value 74AHC1G14 -> 74AHC1G00
- U20: value 74LS161 -> 74LS21; footprint Package_SO:SOIC-16_3.9x9.9mm_P1.27mm -> Package_SO:SOIC-14_3.9x8.7mm_P1.27mm; moved to B.Cu
- U22, U23, U24: value MC33078 -> LMH6642; footprint Package_SO:SOIC-8_3.9x4.9mm_P1.27mm -> Package_TO_SOT_SMD:SOT-23-5
- U3: value 74AHC1G00 -> 74LS161; footprint Package_TO_SOT_SMD:SOT-23-5 -> Package_SO:SOIC-16_3.9x9.9mm_P1.27mm
- U5: value 74LS161 -> 74AHC04; footprint Package_SO:SOIC-16_3.9x9.9mm_P1.27mm -> Package_SO:SOIC-14_3.9x8.7mm_P1.27mm
- U6: moved to F.Cu
- U7: value 74AHC04 -> 74LS30; moved to F.Cu
- Y1: value 13.5 MHz -> 18 MHz; footprint Crystal:Crystal_SMD_HC49-SD -> Crystal:Crystal_HC49-4H_Vertical
- moved C1 147.7 mm to (95.5, 56.0), turned to 90 degrees
- moved C2 143.1 mm to (103.1, 57.0), turned to 90 degrees
- moved U1 141.2 mm to (100.4, 56.6), turned to -90 degrees
- moved R2 139.0 mm to (110.3, 52.3), turned to 180 degrees
- moved Y1 138.4 mm to (95.6, 59.7), turned to -90 degrees
- moved R1 135.4 mm to (99.5, 61.6), turned to -90 degrees
- moved C5 134.8 mm to (85.0, 48.2), turned to 0 degrees
- moved C4 133.7 mm to (95.6, 67.4)
- moved R3 131.7 mm to (99.5, 64.8)
- moved U15 126.0 mm to (142.2, 94.6)
- moved J1 125.1 mm to (93.7, 84.7)
- moved U12 122.9 mm to (141.9, 72.4), turned to -90 degrees
- moved U2 120.0 mm to (126.7, 101.5), turned to 90 degrees
- moved C13 119.2 mm to (146.9, 97.4), turned to 90 degrees
- moved C12 115.0 mm to (146.9, 86.2), turned to 90 degrees
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Connections:
- C5 pad 1: +5V -> /9mhz
- C6 pad 1: /HCounter/CLK -> +5V
- J3 pad 1: /RAM_ADDR0 -> /5-bit DAC2/AOUT
- J3 pad 2: /RAM_ADDR1 -> /5-bit DAC1/AOUT
- J3 pad 3: /RAM_ADDR2 -> /5-bit DAC/AOUT
- J3 pad 4: /RAM_ADDR3 -> unconnected-(J3-Pad4)
- J3 pad 5: /RAM_ADDR4 -> GND
- J3 pad 6: /RAM_ADDR5 -> GND
- J3 pad 7: /RAM_ADDR6 -> GND
- J3 pad 8: /RAM_ADDR7 -> GND
- J4 pad 1: /5-bit DAC2/AOUT -> /RAM_ADDR0
- J4 pad 10: GND -> /RAM_ADDR9
- J4 pad 11: unconnected-(J4-Pad11) -> /RAM_ADDR10
- J4 pad 12: unconnected-(J4-Pad12) -> /RAM_ADDR11
- J4 pad 13: /h_sync -> /RAM_ADDR12
- J4 pad 14: /v_sync -> /RAM_ADDR13
- J4 pad 15: unconnected-(J4-Pad15) -> /RAM_ADDR14
- J4 pad 2: /5-bit DAC1/AOUT -> /RAM_ADDR1
- J4 pad 3: /5-bit DAC/AOUT -> /RAM_ADDR2
- J4 pad 4: unconnected-(J4-Pad4) -> /RAM_ADDR3
- J4 pad 5: GND -> /RAM_ADDR4
- J4 pad 6: GND -> /RAM_ADDR5
- J4 pad 7: GND -> /RAM_ADDR6
- J4 pad 8: GND -> /RAM_ADDR7
- J4 pad 9: GND -> /RAM_ADDR8
- J5 pad 1: /RAM_ADDR0 -> /MEMIN0
- J5 pad 10: /RAM_ADDR9 -> /MEMIN9
- J5 pad 11: /RAM_ADDR10 -> /MEMIN10
- J5 pad 12: /RAM_ADDR11 -> /MEMIN11
- J5 pad 13: /RAM_ADDR12 -> /MEMIN12
- J5 pad 14: /RAM_ADDR13 -> /MEMIN13
- J5 pad 15: /RAM_ADDR14 -> /MEMIN14
- J5 pad 16: /word_conn/IN15 -> /MEMIN15
- J5 pad 2: /RAM_ADDR1 -> /MEMIN1
- J5 pad 3: /RAM_ADDR2 -> /MEMIN2
- J5 pad 4: /RAM_ADDR3 -> /MEMIN3
- J5 pad 5: /RAM_ADDR4 -> /MEMIN4
- J5 pad 6: /RAM_ADDR5 -> /MEMIN5
- J5 pad 7: /RAM_ADDR6 -> /MEMIN6
- J5 pad 8: /RAM_ADDR7 -> /MEMIN7
- J5 pad 9: /RAM_ADDR8 -> /MEMIN8
- R1 pad 2: Net-(R1-Pad2) -> /18mhz
- R14 pad 1: Net-(U22A--) -> Net-(U22--)
- R14 pad 2: Net-(U22B-+) -> GND
- R15 pad 1: Net-(U22B-+) -> GND
- R15 pad 2: GND -> Net-(R15-Pad2)
- R16 pad 1: /5-bit DAC1/AOUT -> Net-(R15-Pad2)
- R16 pad 2: Net-(U22B--) -> /MEMIN0
- R17 pad 1: GND -> Net-(R15-Pad2)
- R18 pad 2: /MEMIN0 -> /MEMIN1
- R20 pad 2: /MEMIN1 -> /MEMIN2
- R22 pad 2: /MEMIN2 -> /MEMIN3
- R23 pad 2: Net-(R23-Pad2) -> Net-(U23-+)
- R24 pad 1: Net-(R23-Pad2) -> Net-(U23-+)
- R24 pad 2: /MEMIN3 -> /MEMIN4
- R25 pad 1: Net-(R23-Pad2) -> Net-(U23--)
- R25 pad 2: Net-(U23A-+) -> GND
- R26 pad 1: Net-(U23A-+) -> GND
- R26 pad 2: /MEMIN4 -> Net-(R26-Pad2)
- R27 pad 1: Net-(U23A--) -> Net-(R26-Pad2)
- R27 pad 2: Net-(U23B-+) -> /MEMIN10
- R28 pad 1: Net-(U23B-+) -> Net-(R26-Pad2)
- R28 pad 2: GND -> Net-(R28-Pad2)
- R29 pad 1: /5-bit DAC/AOUT -> Net-(R28-Pad2)
- R29 pad 2: Net-(U23B--) -> /MEMIN11
- R3 pad 1: Net-(R1-Pad2) -> /18mhz
- R30 pad 1: GND -> Net-(R28-Pad2)
- R31 pad 2: /MEMIN10 -> /MEMIN12
- R33 pad 2: /MEMIN11 -> /MEMIN13
- R34 pad 2: Net-(R34-Pad2) -> Net-(U24-+)
- R35 pad 1: Net-(R34-Pad2) -> Net-(U24-+)
- R35 pad 2: /MEMIN12 -> /MEMIN14
- R36 pad 1: Net-(R34-Pad2) -> Net-(U24--)
- R36 pad 2: Net-(R36-Pad2) -> GND
- R37 pad 1: Net-(R36-Pad2) -> Net-(U22--)
- R37 pad 2: /MEMIN13 -> /5-bit DAC1/AOUT
- R38 pad 1: Net-(R36-Pad2) -> Net-(U23--)
- R38 pad 2: Net-(U24A-+) -> /5-bit DAC/AOUT
- R39 pad 1: Net-(U24A-+) -> Net-(U24--)
- R39 pad 2: /MEMIN14 -> /5-bit DAC2/AOUT
- TP1 pad 1: /HCounter/CLK -> /9mhz
- U1 pad 1: (no net) -> unconnected-(U1-NC-Pad1)
- U1 pad 4: Net-(R1-Pad2) -> /18mhz
- U10 pad 1: /RAM_ADDR0 -> /RAM_ADDR5
- U10 pad 11: /RAM_ADDR6 -> /HCounter/~{B4}
- U10 pad 12: /RAM_ADDR7 -> /HCounter/~{B6}
- U10 pad 2: /RAM_ADDR1 -> /HCounter/~{B0}
- U10 pad 3: /HCounter/~{B2} -> /RAM_ADDR7
- U10 pad 5: /RAM_ADDR4 -> /HCounter/~{B2}
- U10 pad 6: /HCounter/~{B5} -> /HCounter/~{B1}
- U10 pad 8: /HCounter/~{READ SET} -> /HCounter/~{READ RESET}
- U11 pad 1: /HCounter/~{B0} -> /HCounter/~{SYNC SET}
- U11 pad 10: (no net) -> Net-(U11-Pad10)
- U11 pad 11: /HCounter/~{B6} -> Net-(U11-Pad10)
- U11 pad 12: /RAM_ADDR7 -> /HCounter/OE
- U11 pad 13: (no net) -> /HCounter/~{READ RESET}
- U11 pad 2: /HCounter/~{B1} -> /h_sync
- U11 pad 3: /HCounter/~{B2} -> Net-(U11-Pad3)
- U11 pad 4: /HCounter/~{B3} -> Net-(U11-Pad3)
- U11 pad 5: /HCounter/~{B4} -> /HCounter/~{SYNC RESET}
- U11 pad 6: /RAM_ADDR5 -> /h_sync
- U11 pad 8: /HCounter/~{READ RESET} -> /HCounter/OE
- U11 pad 9: (no net) -> /HCounter/~{READ SET}
- U12 pad 1: /HCounter/~{SYNC SET} -> /VCounter/B0
- U12 pad 10: Net-(U12-Pad10) -> /VCounter/~{B4}
- U12 pad 11: Net-(U12-Pad10) -> /RAM_ADDR10
- U12 pad 12: /HCounter/OE -> (no net)
- U12 pad 13: /HCounter/~{READ RESET} -> (no net)
- U12 pad 14: (no net) -> +5V
- U12 pad 2: /h_sync -> /VCounter/~{B0}
- U12 pad 3: Net-(U12-Pad3) -> /VCounter/B1
- U12 pad 4: Net-(U12-Pad3) -> /VCounter/~{B1}
- U12 pad 5: /HCounter/~{SYNC RESET} -> /RAM_ADDR8
- U12 pad 6: /h_sync -> /VCounter/~{B2}
- U12 pad 7: (no net) -> GND
- U12 pad 8: /HCounter/OE -> /VCounter/~{B3}
- U12 pad 9: /HCounter/~{READ SET} -> /RAM_ADDR9
- U13 pad 1: /VCounter/B0 -> /VCounter/~{B4}
- U13 pad 10: /VCounter/~{B4} -> (no net)
- U13 pad 11: /RAM_ADDR9 -> unconnected-(U13-Pad11)
- U13 pad 12: /VCounter/~{B5} -> unconnected-(U13-Pad12)
- U13 pad 13: /RAM_ADDR10 -> (no net)
- U13 pad 2: /VCounter/~{B0} -> Net-(U13-Pad2)
- U13 pad 3: /VCounter/B1 -> /VCounter/~{B2}
- U13 pad 4: /VCounter/~{B1} -> /VCounter/~{B3}
- U13 pad 5: /VCounter/B2 -> /VCounter/~{B1}
- U13 pad 6: /VCounter/~{B2} -> /VCounter/~{B0}
- U13 pad 8: /VCounter/~{B3} -> /VCounter/~{SYNC SET}
- U13 pad 9: /RAM_ADDR8 -> (no net)
- U14 pad 1: /VCounter/B0 -> /RAM_ADDR8
- U14 pad 11: /VCounter/B10 -> unconnected-(U14-Pad11)
- U14 pad 12: +5V -> unconnected-(U14-Pad12)
- U14 pad 2: /VCounter/~{B1} -> /VCounter/~{B0}
- U14 pad 3: /VCounter/~{B2} -> /VCounter/~{B1}
- U14 pad 5: /VCounter/~{B4} -> Net-(U13-Pad2)
- U14 pad 6: /VCounter/~{B5} -> /VCounter/~{B4}
- U14 pad 8: /VCounter/~{SYNC SET} -> /VCounter/~{SYNC RESET}
- U15 pad 1: /VCounter/~{B0} -> /VCounter/B0
- U15 pad 11: /VCounter/B10 -> unconnected-(U15-Pad11)
- U15 pad 12: +5V -> unconnected-(U15-Pad12)
- U15 pad 2: /VCounter/~{B1} -> /RAM_ADDR10
- U15 pad 3: /VCounter/B2 -> /RAM_ADDR9
- U15 pad 4: /VCounter/~{B3} -> Net-(U13-Pad2)
- U15 pad 5: /VCounter/~{B4} -> /RAM_ADDR8
- U15 pad 6: /VCounter/~{B5} -> unconnected-(U15-Pad6)
- U15 pad 8: /VCounter/~{SYNC RESET} -> /VCounter/~{READ SET}
- U16 pad 11: /VCounter/B10 -> unconnected-(U16-Pad11)
- U16 pad 12: +5V -> unconnected-(U16-Pad12)
- U16 pad 2: /VCounter/B1 -> /VCounter/~{B1}
- U16 pad 3: /VCounter/~{B2} -> /VCounter/~{B3}
- U16 pad 4: /RAM_ADDR8 -> /VCounter/~{B2}
- U16 pad 6: /RAM_ADDR10 -> Net-(U13-Pad2)
- U16 pad 8: /VCounter/~{READ SET} -> /VCounter/~{READ RESET}
- U17 pad 1: /VCounter/~{B0} -> /VCounter/~{READ SET}
- U17 pad 10: (no net) -> +5V
- U17 pad 11: /VCounter/B10 -> /RAM_ADDR9
- U17 pad 12: +5V -> /RAM_ADDR8
- U17 pad 13: (no net) -> /VCounter/B1
- U17 pad 14: +5V -> /VCounter/B0
- U17 pad 2: /VCounter/~{B1} -> /HCounter/~{READ RESET}
- U17 pad 3: /VCounter/~{B2} -> unconnected-(U17-D0-Pad3)
- U17 pad 4: /VCounter/~{B3} -> unconnected-(U17-D1-Pad4)
- U17 pad 5: /VCounter/~{B4} -> unconnected-(U17-D2-Pad5)
- U17 pad 6: /VCounter/~{B5} -> unconnected-(U17-D3-Pad6)
- U17 pad 7: GND -> +5V
- U17 pad 8: /VCounter/~{READ RESET} -> GND
- U17 pad 9: (no net) -> +5V
- U18 pad 10: +5V -> Net-(U17-TC)
- U18 pad 11: /RAM_ADDR8 -> /RAM_ADDR13
- U18 pad 12: /VCounter/B2 -> /RAM_ADDR12
- U18 pad 13: /VCounter/B1 -> /RAM_ADDR11
- U18 pad 14: /VCounter/B0 -> /RAM_ADDR10
- U19 pad 11: /RAM_ADDR12 -> unconnected-(U19-Q3-Pad11)
- U19 pad 12: /RAM_ADDR11 -> unconnected-(U19-Q2-Pad12)
- U19 pad 13: /RAM_ADDR10 -> unconnected-(U19-Q1-Pad13)
- U19 pad 14: /RAM_ADDR9 -> /RAM_ADDR14
- U19 pad 15: Net-(U19-TC) -> unconnected-(U19-TC-Pad15)
- U2 pad 1: unconnected-(U2-NC-Pad1) -> /HCounter/OE
- U2 pad 2: Net-(R1-Pad2) -> /VCounter/OE
- U2 pad 4: /HCounter/CLK -> /~{OE}
- U20 pad 1: /VCounter/~{READ SET} -> /RAM_ADDR14
- U20 pad 10: Net-(U19-TC) -> (no net)
- U20 pad 11: unconnected-(U20-Q3-Pad11) -> (no net)
- U20 pad 12: /VCounter/B10 -> (no net)
- U20 pad 13: /RAM_ADDR14 -> (no net)
- U20 pad 14: /RAM_ADDR13 -> +5V
- U20 pad 2: /HCounter/~{READ RESET} -> /RAM_ADDR11
- U20 pad 3: unconnected-(U20-D0-Pad3) -> (no net)
- U20 pad 4: unconnected-(U20-D1-Pad4) -> /RAM_ADDR12
- U20 pad 5: unconnected-(U20-D2-Pad5) -> /RAM_ADDR13
- U20 pad 6: unconnected-(U20-D3-Pad6) -> Net-(U13-Pad2)
- U20 pad 7: +5V -> GND
- U20 pad 8: GND -> (no net)
- U20 pad 9: +5V -> (no net)
- U22 pad 1: Net-(U22A--) -> Net-(U22--)
- U22 pad 2: Net-(U22A--) -> GND
- U22 pad 4: GND -> Net-(U22--)
- U22 pad 5: Net-(U22B-+) -> +5V
- U23 pad 1: Net-(U23A--) -> Net-(U23--)
- U23 pad 2: Net-(U23A--) -> GND
- U23 pad 3: Net-(U23A-+) -> Net-(U23-+)
- U23 pad 4: GND -> Net-(U23--)
- U23 pad 5: Net-(U23B-+) -> +5V
- U24 pad 1: Net-(U24A--) -> Net-(U24--)
- U24 pad 2: Net-(U24A--) -> GND
- U24 pad 3: Net-(U24A-+) -> Net-(U24-+)
- U24 pad 4: GND -> Net-(U24--)
- U24 pad 5: Net-(U24B-+) -> +5V
- U3 pad 1: /HCounter/OE -> /HCounter/~{READ RESET}
- U3 pad 2: /VCounter/OE -> /9mhz
- U3 pad 3: GND -> unconnected-(U3-D0-Pad3)
- U3 pad 4: /~{OE} -> unconnected-(U3-D1-Pad4)
- U3 pad 5: +5V -> unconnected-(U3-D2-Pad5)
- U4 pad 10: +5V -> Net-(U3-TC)
- U4 pad 11: /RAM_ADDR3 -> /RAM_ADDR7
- U4 pad 12: /RAM_ADDR2 -> /RAM_ADDR6
- U4 pad 13: /RAM_ADDR1 -> /RAM_ADDR5
- U4 pad 14: /RAM_ADDR0 -> /RAM_ADDR4
- U4 pad 15: Net-(U4-TC) -> unconnected-(U4-TC-Pad15)
- U4 pad 2: /HCounter/CLK -> /9mhz
- U5 pad 1: /HCounter/~{READ RESET} -> /RAM_ADDR4
- U5 pad 10: Net-(U4-TC) -> /HCounter/~{B0}
- U5 pad 11: /RAM_ADDR7 -> /RAM_ADDR0
- U5 pad 12: /RAM_ADDR6 -> (no net)
- U5 pad 13: /RAM_ADDR5 -> (no net)
- U5 pad 14: /RAM_ADDR4 -> +5V
- U5 pad 2: /HCounter/CLK -> /HCounter/~{B4}
- U5 pad 3: unconnected-(U5-D0-Pad3) -> /RAM_ADDR5
- U5 pad 4: unconnected-(U5-D1-Pad4) -> /HCounter/~{B5}
- U5 pad 5: unconnected-(U5-D2-Pad5) -> /RAM_ADDR6
- U5 pad 6: unconnected-(U5-D3-Pad6) -> /HCounter/~{B6}
- U5 pad 7: +5V -> GND
- U5 pad 8: GND -> (no net)
- U5 pad 9: +5V -> (no net)
- U6 pad 1: /RAM_ADDR0 -> /RAM_ADDR1
- U6 pad 2: /HCounter/~{B0} -> /HCounter/~{B1}
- U6 pad 3: /RAM_ADDR1 -> /RAM_ADDR2
- U6 pad 4: /HCounter/~{B1} -> /HCounter/~{B2}
- U6 pad 5: /RAM_ADDR2 -> /RAM_ADDR3
- U6 pad 6: /HCounter/~{B2} -> /HCounter/~{B3}
- U6 pad 8: /HCounter/~{B3} -> Net-(U25-Pad4)
- U6 pad 9: /RAM_ADDR3 -> Net-(U25-Pad1)
- U7 pad 1: /RAM_ADDR4 -> /HCounter/~{B2}
- U7 pad 11: (no net) -> /RAM_ADDR3
- U7 pad 12: (no net) -> /HCounter/~{B4}
- U7 pad 2: /HCounter/~{B4} -> /RAM_ADDR7
- U7 pad 4: /HCounter/~{B5} -> /HCounter/~{B6}
- U7 pad 5: /RAM_ADDR6 -> /HCounter/~{B0}
- U7 pad 6: /HCounter/~{B6} -> /HCounter/~{B1}
- U7 pad 8: /HCounter/~{B7} -> /HCounter/~{SYNC SET}
- U7 pad 9: /RAM_ADDR7 -> (no net)
- U8 pad 1: /RAM_ADDR5 -> /HCounter/~{B1}
- U8 pad 11: /HCounter/~{B6} -> /RAM_ADDR4
- U8 pad 12: /RAM_ADDR7 -> /RAM_ADDR2
- U8 pad 2: /HCounter/~{B4} -> /HCounter/~{B0}
- U8 pad 3: /RAM_ADDR2 -> /HCounter/~{B6}
- U8 pad 4: /HCounter/~{B3} -> /RAM_ADDR5
- U8 pad 5: /RAM_ADDR1 -> /RAM_ADDR7
- U8 pad 6: /HCounter/~{B0} -> /HCounter/~{B3}
- U8 pad 8: /HCounter/~{SYNC SET} -> /HCounter/~{SYNC RESET}
- U9 pad 1: /HCounter/~{B0} -> /HCounter/~{B5}
- U9 pad 11: /HCounter/~{B6} -> /RAM_ADDR6
- U9 pad 12: /RAM_ADDR7 -> /RAM_ADDR4
- U9 pad 3: /RAM_ADDR2 -> /HCounter/~{B2}
- U9 pad 5: /RAM_ADDR4 -> /RAM_ADDR7
- U9 pad 6: /RAM_ADDR5 -> /HCounter/~{B0}
- U9 pad 8: /HCounter/~{SYNC RESET} -> /HCounter/~{READ SET}
Routing:
- net /HCounter/~{READ RESET}: track 0.00 -> 104.6 mm, vias 0 -> 7
- net +5V: track 6.69 -> 111.3 mm, vias 2 -> 25
- net /VCounter/~{READ SET}: track 0.00 -> 88.0 mm, vias 0 -> 4
- net GND: track 23.3 -> 108.8 mm, vias 1 -> 43
- net /h_sync: track 0.00 -> 81.2 mm
- net /RAM_ADDR9: track 0.00 -> 59.2 mm, vias 0 -> 3
- net /RAM_ADDR8: track 0.00 -> 58.5 mm, vias 0 -> 3
- net /RAM_ADDR10: track 0.00 -> 56.1 mm, vias 0 -> 4
- net /9mhz: track 0.00 -> 50.1 mm, vias 0 -> 3
- net /v_sync: track 0.00 -> 46.4 mm, vias 0 -> 1
- net Net-(U13-Pad2): track 0.00 -> 43.6 mm, vias 0 -> 2
- net /VCounter/B0: track 0.00 -> 40.5 mm, vias 0 -> 2
- net /HCounter/~{B1}: track 0.00 -> 39.5 mm, vias 0 -> 2
- net /RAM_ADDR6: track 14.8 -> 54.2 mm, vias 1 -> 3
- net /HCounter/~{B0}: track 4.53 -> 41.6 mm, vias 1 -> 2
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Other:
- board outline added: 82 x 60 mm

Commit message: updated gpu
Parts:
- removed C5: 50 pF, Capacitor_SMD:C_0603_1608Metric
- removed U1: 74AHC1G14, Package_TO_SOT_SMD:SOT-23-5
- removed U25: 74HC00, Package_SO:SOIC-14_3.9x8.7mm_P1.27mm
- removed Y1: 18 MHz, Crystal:Crystal_HC49-4H_Vertical
- added C28: 0.1uF, Capacitor_SMD:C_0603_1608Metric, B.Cu at (104.0, 65.2)
- added C29: 0.1uF, Capacitor_SMD:C_0603_1608Metric, B.Cu at (109.2, 65.2)
- added C30: 0.1uF, Capacitor_SMD:C_0603_1608Metric, F.Cu at (125.6, 63.2)
- added D2: LED_Small, LED_SMD:LED_0603_1608Metric, F.Cu at (101.6, 55.6)
- added D3: LED_Small, LED_SMD:LED_0603_1608Metric, F.Cu at (151.2, 94.4)
- added D4: LED_Small, LED_SMD:LED_0603_1608Metric, F.Cu at (128.4, 106.4)
- added D5: LED_Small, LED_SMD:LED_0603_1608Metric, F.Cu at (156.4, 107.2)
- added D6: LED_Small, LED_SMD:LED_0603_1608Metric, F.Cu at (156.6, 102.6)
- added J6: Conn_01x01, Connector_PinHeader_2.54mm:PinHeader_1x01_P2.54mm_Vertical, F.Cu at (93.7, 73.2)
- added J7: Conn_Coaxial, Connector_Coaxial:SMA_Amphenol_132289_EdgeMount, F.Cu at (93.8, 64.5)
- added R40: 220, Resistor_SMD:R_0603_1608Metric, F.Cu at (132.2, 106.4)
- added R41: 220, Resistor_SMD:R_0603_1608Metric, F.Cu at (153.2, 107.2)
- added R42: 220, Resistor_SMD:R_0603_1608Metric, F.Cu at (153.2, 102.6)
- added TP10: TestPoint, TestPoint:TestPoint_Pad_D2.0mm, F.Cu at (131.9, 101.7)
- added TP11: NEW FRAME, TestPoint:TestPoint_Pad_D2.0mm, F.Cu at (150.4, 89.2)
- added TP9: TestPoint, TestPoint:TestPoint_Pad_D2.0mm, F.Cu at (120.5, 103.1)
- C1, C4: value 36 pF -> 100 pF; moved to F.Cu
- C2: value 0.1uF -> 100 pF
- R1: value 1M -> 220
- R14: footprint Resistor_SMD:R_0603_1608Metric -> Resistor_SMD:R_0402_1005Metric; moved to B.Cu
- R25, R36: footprint Resistor_SMD:R_0603_1608Metric -> Resistor_SMD:R_0402_1005Metric
- R3: value 1k -> 220
- U10, U13, U14, U15, U16, U7, U8, U9: value 74LS30 -> 74HC30
- U17, U18, U19, U3, U4: value 74LS161 -> 74HC161
- U20: value 74LS21 -> 74HC21
- moved C1 71.7 mm to (166.0, 68.9), turned to 0 degrees
- moved C4 63.1 mm to (158.5, 71.2), turned to 0 degrees
- moved R3 58.6 mm to (151.2, 92.4), turned to 0 degrees
- moved C2 50.8 mm to (151.3, 73.1), turned to 0 degrees
- moved R1 8.21 mm to (105.2, 55.6), turned to 180 degrees
- moved TP1 6.04 mm to (97.3, 75.6)
- moved R14 4.04 mm to (159.2, 66.9), turned to 180 degrees
- moved C24 3.81 mm to (151.3, 74.7)
- moved R36 3.79 mm to (170.0, 62.2)
- moved R25 3.34 mm to (153.3, 67.6), turned to 180 degrees
- moved TP7 2.92 mm to (169.5, 72.7)
- moved TP8 2.60 mm to (154.9, 85.5)
- moved U23 2.47 mm to (151.9, 70.6)
- moved C23 2.31 mm to (158.5, 72.8)
- moved TP6 1.90 mm to (159.9, 83.8)
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Connections:
- C1 pad 1: Net-(C1-Pad1) -> +5V
- C4 pad 1: Net-(C4-Pad1) -> +5V
- R1 pad 1: Net-(C1-Pad1) -> /HCounter/~{READ SET}
- R1 pad 2: /18mhz -> Net-(D2-A)
- R14 pad 1: Net-(U22--) -> Net-(U22-+)
- R25 pad 1: Net-(U23--) -> Net-(U23-+)
- R3 pad 1: /18mhz -> /VCounter/~{READ SET}
- R3 pad 2: Net-(C4-Pad1) -> Net-(D3-A)
- R36 pad 1: Net-(U24--) -> Net-(U24-+)
- TP2 pad 1: /HCounter/~{READ RESET} -> /HCounter/~{READ SET}
- U13 pad 11: unconnected-(U13-Pad11) -> +5V
- U13 pad 12: unconnected-(U13-Pad12) -> +5V
- U13 pad 6: /VCounter/~{B0} -> /VCounter/B0
- U14 pad 11: unconnected-(U14-Pad11) -> +5V
- U14 pad 12: unconnected-(U14-Pad12) -> +5V
- U15 pad 11: unconnected-(U15-Pad11) -> +5V
- U15 pad 12: unconnected-(U15-Pad12) -> +5V
- U15 pad 6: unconnected-(U15-Pad6) -> /VCounter/~{B1}
- U16 pad 11: unconnected-(U16-Pad11) -> +5V
- U16 pad 12: unconnected-(U16-Pad12) -> +5V
- U17 pad 2: /HCounter/~{READ RESET} -> /HCounter/~{READ SET}
- U17 pad 3: unconnected-(U17-D0-Pad3) -> GND
- U17 pad 4: unconnected-(U17-D1-Pad4) -> GND
- U17 pad 5: unconnected-(U17-D2-Pad5) -> GND
- U17 pad 6: unconnected-(U17-D3-Pad6) -> GND
- U18 pad 2: /HCounter/~{READ RESET} -> /HCounter/~{READ SET}
- U18 pad 3: unconnected-(U18-D0-Pad3) -> GND
- U18 pad 4: unconnected-(U18-D1-Pad4) -> GND
- U18 pad 5: unconnected-(U18-D2-Pad5) -> GND
- U18 pad 6: unconnected-(U18-D3-Pad6) -> GND
- U19 pad 2: /HCounter/~{READ RESET} -> /HCounter/~{READ SET}
- U19 pad 3: unconnected-(U19-D0-Pad3) -> GND
- U19 pad 4: unconnected-(U19-D1-Pad4) -> GND
- U19 pad 5: unconnected-(U19-D2-Pad5) -> GND
- U19 pad 6: unconnected-(U19-D3-Pad6) -> GND
- U3 pad 1: /HCounter/~{READ RESET} -> /HCounter/~{READ SET}
- U3 pad 3: unconnected-(U3-D0-Pad3) -> GND
- U3 pad 4: unconnected-(U3-D1-Pad4) -> GND
- U3 pad 5: unconnected-(U3-D2-Pad5) -> GND
- U3 pad 6: unconnected-(U3-D3-Pad6) -> GND
- U4 pad 1: /HCounter/~{READ RESET} -> /HCounter/~{READ SET}
- U4 pad 3: unconnected-(U4-D0-Pad3) -> GND
- U4 pad 4: unconnected-(U4-D1-Pad4) -> GND
- U4 pad 5: unconnected-(U4-D2-Pad5) -> GND
- U4 pad 6: unconnected-(U4-D3-Pad6) -> GND
- U6 pad 8: Net-(U25-Pad4) -> (no net)
- U6 pad 9: Net-(U25-Pad1) -> (no net)
- U7 pad 1: /HCounter/~{B2} -> /RAM_ADDR2
- U7 pad 11: /RAM_ADDR3 -> /RAM_ADDR1
- U7 pad 6: /HCounter/~{B1} -> /RAM_ADDR3
- U8 pad 1: /HCounter/~{B1} -> /RAM_ADDR3
- U8 pad 12: /RAM_ADDR2 -> /HCounter/~{B1}
- U8 pad 6: /HCounter/~{B3} -> /RAM_ADDR2
Routing:
- net /HCounter/~{READ SET}: track 9.16 -> 109.7 mm, vias 0 -> 6
- net /HCounter/~{READ RESET}: track 104.6 -> 17.9 mm, vias 7 -> 2
- net +5V: track 111.3 -> 144.4 mm, vias 25 -> 29
- net /18mhz: track 32.0 -> 0.00 mm
- net Net-(U25-Pad1): track 25.5 -> 0.00 mm, vias 3 -> 0
- net /RAM_ADDR1: track 23.5 -> 47.2 mm, vias 1 -> 2
- net Net-(C1-Pad1): track 18.6 -> 0.00 mm
- net Net-(U25-Pad4): track 16.2 -> 0.00 mm, vias 2 -> 0
- net /RAM_ADDR2: track 50.8 -> 60.3 mm, vias 2 -> 4
- net /HCounter/~{B3}: track 43.5 -> 35.3 mm
- net /RAM_ADDR3: track 45.2 -> 52.9 mm, vias 0 -> 4
- net /~{OE}: track 9.19 -> 16.9 mm
- net GND: track 108.8 -> 101.2 mm, vias 43 -> 55
- net /VCounter/~{B1}: track 33.6 -> 40.3 mm
- net /VCounter/B0: track 40.5 -> 47.1 mm, vias 2 -> 3
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Other:
- board size 82 x 60 mm -> 81 x 60 mm
- board text added: "+5V"
- board text added: "0"
- board text added: "1"
- board text added: "15"
- board text added: "1k"
- board text added: "2k"
- board text added: "9MHz"
- board text added: "ADDR"
- board text added: "B"
- board text added: "G"
- board text added: "GND"
- board text added: "GPU"
- board text added: "H_{SYNC}"
- board text added: "IO"
- board text added: "NEW FRAME"
- board text added: "NEW LINE"
- board text added: "PWR"
- board text added: "R"
- board text added: "V1.0"
- board text added: "V_{SYNC}"
- board text added: "~{H_{OE}}"
- board text added: "~{OE}"
- board text added: "~{V_{OE}}"
